File: hardware/CPU_board/untitled.brd (EAGLE design)
At the start: 109.2 x 94.3 mm, 31 parts, among them IC1 MAX232ECWE, IC2 MAX232ECWE, IC3 AM29F040J, IC5 LM2596S, J2 POWER_JACKSLT, U1 AS6C4008-55SIN

Commit message: PCB updated
Connections:
- removed net VCC: IC3.32
- net 5V: now also IC3.32
Routing:
- net A15: track 0.00 -> 33.8 mm
- net D3: track 0.00 -> 31.6 mm
- net !WR: track 0.00 -> 30.2 mm
- net D1: track 0.00 -> 24.1 mm
- net D2: track 0.00 -> 23.1 mm
- net A0: track 9.18 -> 29.8 mm
- net A16: track 0.00 -> 20.5 mm
- net A18: track 0.00 -> 17.2 mm
- net !ROM_CS: track 0.00 -> 15.4 mm, vias 0 -> 1
- net 5V: track 16.4 -> 18.5 mm, vias 0 -> 1
- net D0: track 23.3 -> 24.3 mm
- net D4: track 28.7 -> 29.6 mm

Commit message: PCB project updated (work in progress)
Parts:
- removed U$2: PINHD-2X40, pinhead:2X40
- added C13, C14: (no value), rcl:C0603
- added C15, C16: 22 pF, rcl:C0603
- added JP1: (no value), pinhead:1X12
- added JP3: (no value), pinhead:1X20
- added Y1: CRYSTAL-GROUNDEDSMD-5X3.2, SparkFun-Clocks:CRYSTAL-SMD-5X3.2-4PAD
- moved IC3 51.4 mm to (101.3, 27.2)
- moved U1 51.4 mm to (81.0, 28.5)
- moved C2 21.9 mm to (42.1, 43.5)
- moved C3 21.1 mm to (55.6, 36.0)
- moved U$1 21.1 mm to (44.8, 33.5)
- moved C1 17.5 mm to (52.4, 23.5), turned to 0 degrees
Connections:
- removed net !BAK: U$2.44
- removed net !BRQ: U$2.48
- removed net !MRQ: U$2.45
- removed net A20: U$2.24
- removed net A21: U$2.22
- removed net A22: U$2.20
- removed net A23: U$2.18
- removed net BAI: U$2.4
- removed net BAO: U$2.6
- removed net CLK2: U$2.42
- removed net D10: U$2.58
- removed net D11: U$2.60
- removed net D12: U$2.62
- removed net D13: U$2.64
- removed net D14: U$2.66
- removed net D15: U$2.68
- removed net D8: U$2.54
- removed net D9: U$2.56
- removed net P41: U$2.2
- removed net P44: U$2.8
- removed net P45: U$2.10
- removed net P46: U$2.12
- removed net P47: U$2.14
- removed net P48: U$2.16
- removed net P78: U$2.76
- removed net P79: U$2.78
- removed net PAGE: U$2.40
- removed net RX2: U$2.72
- removed net TX2: U$2.70
- removed net USR8: U$2.80
- new net !MRQ_NOT_CONNECTED: JP3.18
- new net OSC_IN: C16.1, U$1.91, Y1.1
- new net OSC_OUT: C15.1, U$1.92, Y1.3
- net !HLT: no longer U$2.46
- net !INT: now also JP3.19; no longer U$2.43
- net !IORQ: now also JP3.15; no longer U$2.51
- net !IRQ1: now also JP3.4; no longer U$2.73
- net !IRQ2: no longer U$2.74
- net !M1: now also JP1.2; no longer U$2.37
- net !NMI: no longer U$2.52
- net !RD: now also JP3.16; no longer U$1.87, U$2.49
- net !RFSH: no longer U$2.38
- net !RST: now also JP1.1; no longer U$2.39
- net !WAIT: no longer U$2.50
- net !WR: now also JP3.17, U$1.87; no longer U$2.47
- net 5V: now also C13.1, C14.1, JP1.3; no longer U$2.35, U$2.36
- net A0: now also JP1.5; no longer U$2.31
- net A1: now also JP1.6; no longer U$2.29
- net A10: no longer U$2.11
- net A11: no longer U$2.9
- net A12: no longer U$2.7
- net A13: no longer U$2.5
- net A14: no longer U$2.3
- net A15: no longer U$2.1
- net A16: no longer U$2.32
- net A17: no longer U$2.30
- net A18: no longer U$2.28
- net A19: no longer U$2.26
- net A2: now also JP1.7; no longer U$2.27
- net A3: now also JP1.8; no longer U$2.25
- net A4: now also JP1.9; no longer U$2.23
- net A5: now also JP1.10; no longer U$2.21
- net A6: now also JP1.11; no longer U$2.19
- net A7: now also JP1.12; no longer U$2.17
- net A8: no longer U$2.15
- net A9: no longer U$2.13
- net CLK: now also JP3.20; no longer U$2.41
- net D0: now also JP3.14; no longer U$2.53
- net D1: now also JP3.13; no longer U$2.55
- net D2: now also JP3.12; no longer U$2.57
- net D3: now also JP3.11; no longer U$2.59
- net D4: now also JP3.10; no longer U$2.61
- net D5: now also JP3.9; no longer U$2.63
- net D6: now also JP3.8; no longer U$2.65
- net D7: now also JP3.7; no longer U$2.67
- net GND: now also C13.2, C14.2, C15.2, C16.2, JP1.4, Y1.2, Y1.4; no longer U$2.33, U$2.34
- net IEI: now also JP3.3; no longer U$2.75
- net IEO: now also JP3.2; no longer U$2.77
- net RX: now also JP3.5; no longer U$2.71
- net TX: now also JP3.6; no longer U$2.69
- net USR4: now also JP3.1; no longer U$2.79
Routing:
- net !WR: track 30.2 -> 131.4 mm, vias 0 -> 2
- net !IORQ: track 0.00 -> 100.3 mm
- net !IRQ1: track 0.00 -> 100.1 mm, vias 0 -> 1
- net !RD: track 21.5 -> 112.5 mm, vias 0 -> 1
- net !M1: track 0.00 -> 77.5 mm, vias 0 -> 1
- net !INT: track 0.00 -> 62.1 mm
- net !RST: track 0.00 -> 57.3 mm
- net RTS1: track 3.35 -> 57.1 mm
- net CTS1: track 2.08 -> 55.4 mm
- net A0: track 29.8 -> 82.1 mm
- net A14: track 8.23 -> 58.0 mm, vias 0 -> 2
- net A1: track 29.1 -> 75.7 mm
- net RXD1: track 3.35 -> 46.3 mm
- net TXD1: track 2.08 -> 43.9 mm
- net RTS2: track 3.35 -> 44.9 mm
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Other:
- board size 109.2 x 94.3 mm -> 116.8 x 94.9 mm

Commit message: PBC project updated (work in progress)
Connections:
- net CLK: now also U$1.89
Routing:
- net CLK: track 0.00 -> 93.7 mm
- net !WR: track 131.4 -> 144.7 mm
- net !RD: track 112.5 -> 116.8 mm, vias 1 -> 0
- net !IORQ: track 100.3 -> 102.9 mm
- net !M1: track 77.5 -> 79.2 mm
- net !IRQ1: track 100.1 -> 99.3 mm

Commit message: PCB update (work in progress)
Parts:
- moved C13 5.72 mm to (100.1, 26.6)
- moved IC3 5.72 mm to (101.3, 32.9)
- moved C14 5.71 mm to (74.3, 22.5)
- moved U1 5.71 mm to (81.0, 34.2)
Routing:
- net A8: track 32.1 -> 122.3 mm, vias 0 -> 2
- net A5: track 36.2 -> 122.6 mm
- net A6: track 39.1 -> 122.0 mm
- net A7: track 40.8 -> 118.9 mm
- net A12: track 43.3 -> 111.8 mm
- net A9: track 31.6 -> 92.1 mm, vias 0 -> 1
- net D6: track 31.3 -> 75.6 mm, vias 0 -> 1
- net D5: track 33.5 -> 70.0 mm, vias 0 -> 2
- net A10: track 31.0 -> 56.8 mm, vias 0 -> 1
- net A17: track 53.6 -> 28.7 mm
- net A11: track 30.6 -> 54.5 mm, vias 0 -> 1
- net A13: track 29.5 -> 50.4 mm
- net A18: track 40.6 -> 23.6 mm, vias 2 -> 0
- net A16: track 45.6 -> 28.9 mm, vias 1 -> 0
- net D1: track 50.4 -> 38.7 mm, vias 0 -> 1
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
Commit message: PCB update (work in progress)
Parts:
- moved U1 1.91 mm to (81.0, 36.1)
- moved C13 1.90 mm to (100.1, 28.5)
- moved C14 1.90 mm to (74.3, 24.4)
- moved IC3 1.90 mm to (101.3, 34.8)
- moved JP1 1.17 mm to (50.8, 8.99)
- moved JP3 1.17 mm to (91.4, 8.99)
Routing:
- net A0: track 86.1 -> 176.3 mm
- net A3: track 44.3 -> 134.4 mm
- net A4: track 38.0 -> 126.3 mm
- net A1: track 70.7 -> 146.2 mm
- net A2: track 67.3 -> 138.3 mm
- net A16: track 28.9 -> 77.4 mm, vias 0 -> 2
- net A18: track 23.6 -> 68.1 mm, vias 0 -> 2
- net !RD: track 116.8 -> 149.9 mm, vias 0 -> 1
- net A17: track 28.7 -> 60.4 mm, vias 0 -> 2
- net A14: track 49.9 -> 71.1 mm, vias 1 -> 2
- net !WR: track 140.2 -> 161.3 mm, vias 0 -> 2
- net A15: track 69.2 -> 88.2 mm, vias 0 -> 2
- net A10: track 56.8 -> 75.5 mm, vias 1 -> 2
- net A11: track 54.5 -> 73.1 mm, vias 1 -> 2
- net A12: track 111.8 -> 94.4 mm
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
Commit message: PCB update
Routing:
- net A9: track 90.3 -> 122.2 mm, vias 1 -> 2
- net D0: track 49.0 -> 73.8 mm, vias 2 -> 4
- net A0: track 176.3 -> 152.4 mm
- net D6: track 78.7 -> 94.3 mm, vias 1 -> 3
- net D7: track 36.4 -> 50.7 mm
- net !ROM_CS: track 16.0 -> 9.18 mm, vias 1 -> 0
- net D5: track 73.1 -> 71.2 mm, vias 2 -> 3
- net D2: track 37.3 -> 36.1 mm
- net A5: track 123.3 -> 124.5 mm
- net A3: track 134.4 -> 135.4 mm
- net A4: track 126.3 -> 127.3 mm
- net A2: track 138.3 -> 139.2 mm
- net A1: track 146.2 -> 145.4 mm
- net D4: track 33.8 -> 33.1 mm
- net D1: track 38.7 -> 38.1 mm
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
Commit message: Minor update in PCB design
Connections:
- net !WR: no longer IC3.31
- net 5V: now also IC3.31
Routing:
- net D7: track 50.7 -> 83.5 mm
- net !WR: track 161.3 -> 131.2 mm, vias 2 -> 1
- net D1: track 38.1 -> 47.5 mm
- net D5: track 71.2 -> 79.7 mm
- net D4: track 33.1 -> 41.0 mm
- net D0: track 73.8 -> 80.6 mm
- net A18: track 68.0 -> 64.9 mm, vias 2 -> 0
- net D2: track 36.1 -> 33.2 mm
- net D3: track 35.0 -> 32.7 mm
- net 5V: track 29.4 -> 30.7 mm
- net A15: track 88.2 -> 89.0 mm
- net A3: track 135.4 -> 134.7 mm
- net A17: track 60.4 -> 59.7 mm
- net A13: track 67.6 -> 66.9 mm

Commit message: PCB update (work in progress)
Parts:
- moved U1 0.64 mm to (80.4, 36.1)
- moved C14 0.63 mm to (73.7, 24.4)
Routing:
- net D3: track 32.7 -> 86.8 mm
- net D2: track 33.2 -> 86.0 mm
- net D1: track 47.5 -> 97.5 mm
- net D4: track 41.0 -> 79.9 mm
- net D7: track 83.5 -> 50.7 mm
- net A15: track 89.0 -> 86.3 mm
- net A16: track 78.0 -> 76.4 mm
- net A14: track 71.1 -> 72.1 mm
- net !RD: track 149.9 -> 150.8 mm
- net A3: track 134.7 -> 135.3 mm
- net A1: track 145.4 -> 146.0 mm
- net A7: track 119.6 -> 120.2 mm
- net A5: track 124.5 -> 125.1 mm
- net A4: track 127.3 -> 127.9 mm
- net A12: track 94.3 -> 94.9 mm
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