File: hardware/CPU_board/untitled.sch (EAGLE design)
At the start: 64 parts, among them IC1 MAX232ECWE, IC2 MAX232ECWE, IC3 AM29F040J, IC4 74HCT138D, IC5 LM2596S, J2 POWER_JACKSLT, U1 AS6C4008-55SIN, Y1 CRYSTAL-GROUNDEDSMD-5X3.2

Commit message: Buffer added on printer port data lines
Parts:
- added IC6: 74245SSOP, 74xx-eu:74245SSOP
Connections:
- net 5V: now also IC6P.VCC
- net GND: now also IC6A.DIR, IC6A.G, IC6P.GND
- net PD0: now also IC6A.A1
- net PD0_IN: now also IC6A.B1
- net PD1: now also IC6A.A2
- net PD1_IN: now also IC6A.B2
- net PD2: now also IC6A.A3
- net PD2_IN: now also IC6A.B3
- net PD3: now also IC6A.A4
- net PD3_IN: now also IC6A.B4
- net PD4: now also IC6A.A5
- net PD4_IN: now also IC6A.B5
- net PD5: now also IC6A.A6
- net PD5_IN: now also IC6A.B6
- net PD6: now also IC6A.A7
- net PD6_IN: now also IC6A.B7
- net PD7: now also IC6A.A8
- net PD7_IN: now also IC6A.B8
Changed lines of the file:
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@@
 <part name="JP8" library="pinhead" deviceset="PINHD-1X2" device=""/>
 <part name="JP9" library="pinhead-2" deviceset="PINHD-2X13" device="_2.54-SMD"/>
+<part name="IC6" library="74xx-eu" deviceset="74*245" device="SSOP" value="74245SSOP"/>
+<part name="GND22" library="supply1" deviceset="GND" device=""/>
 </parts>
 <sheets>
@@
 <instance part="JP8" gate="G$1" x="-248.92" y="284.48" rot="R90"/>
 <instance part="JP9" gate="A" x="454.66" y="274.32"/>
+<instance part="IC6" gate="A" x="378.46" y="256.54"/>
+<instance part="GND22" gate="1" x="363.22" y="238.76"/>
+<instance part="IC6" gate="P" x="15.24" y="190.5"/>
 </instances>
 <busses>
@@
 <wire x1="5.08" y1="180.34" x2="5.08" y2="182.88" width="0.1524" layer="91"/>
 <junction x="-5.08" y="180.34"/>
+<pinref part="IC6" gate="P" pin="GND"/>
+<wire x1="5.08" y1="180.34" x2="15.24" y2="180.34" width="0.1524" layer="91"/>
+<wire x1="15.24" y1="180.34" x2="15.24" y2="182.88" width="0.1524" layer="91"/>
+<junction x="5.08" y="180.34"/>
 </segment>
 <segment>
@@
 <label x="469.9" y="264.16" size="1.4224" layer="95" xref="yes"/>
 </segment>
+<segment>
+<pinref part="IC6" gate="A" pin="DIR"/>
+<pinref part="GND22" gate="1" pin="GND"/>
+<wire x1="365.76" y1="246.38" x2="363.22" y2="246.38" width="0.1524" layer="91"/>
+<wire x1="363.22" y1="246.38" x2="363.22" y2="243.84" width="0.1524" layer="91"/>
+<pinref part="IC6" gate="A" pin="G"/>
+<wire x1="363.22" y1="243.84" x2="363.22" y2="241.3" width="0.1524" layer="91"/>
+<wire x1="365.76" y1="243.84" x2="363.22" y2="243.84" width="0.1524" layer="91"/>
+<junction x="363.22" y="243.84"/>
+</segment>
 </net>
 <net name="5V" class="0">
@@
 <wire x1="5.08" y1="200.66" x2="5.08" y2="198.12" width="0.1524" layer="91"/>
 <junction x="-5.08" y="200.66"/>
+<pinref part="IC6" gate="P" pin="VCC"/>
+<wire x1="5.08" y1="200.66" x2="15.24" y2="200.66" width="0.1524" layer="91"/>
+<wire x1="15.24" y1="200.66" x2="15.24" y2="198.12" width="0.1524" layer="91"/>
+<junction x="5.08" y="200.66"/>
 </segment>
 <segment>
@@
 <label x="441.96" y="287.02" size="1.4224" layer="95" rot="R180" xref="yes"/>
 </segment>
+<segment>
+<pinref part="IC6" gate="A" pin="A1"/>
+<wire x1="365.76" y1="269.24" x2="360.68" y2="269.24" width="0.1524" layer="91"/>
+<label x="360.68" y="269.24" size="1.4224" layer="95" rot="R180" xref="yes"/>
+</segment>
 </net>
 <net name="PD1" class="0">
@@
 <label x="441.96" y="284.48" size="1.4224" layer="95" rot="R180" xref="yes"/>
 </segment>
+<segment>
+<pinref part="IC6" gate="A" pin="A2"/>
+<wire x1="365.76" y1="266.7" x2="360.68" y2="266.7" width="0.1524" layer="91"/>
+<label x="360.68" y="266.7" size="1.4224" layer="95" rot="R180" xref="yes"/>
+</segment>
 </net>
 <net name="PD2" class="0">
@@
 <label x="441.96" y="281.94" size="1.4224" layer="95" rot="R180" xref="yes"/>
 </segment>
+<segment>
+<pinref part="IC6" gate="A" pin="A3"/>
+<wire x1="365.76" y1="264.16" x2="360.68" y2="264.16" width="0.1524" layer="91"/>
+<label x="360.68" y="264.16" size="1.4224" layer="95" rot="R180" xref="yes"/>
+</segment>
 </net>
 <net name="PD3" class="0">
@@
 <label x="441.96" y="279.4" size="1.4224" layer="95" rot="R180" xref="yes"/>
 </segment>
+<segment>
+<pinref part="IC6" gate="A" pin="A4"/>
+<wire x1="365.76" y1="261.62" x2="360.68" y2="261.62" width="0.1524" layer="91"/>
+<label x="360.68" y="261.62" size="1.4224" layer="95" rot="R180" xref="yes"/>
+</segment>
 </net>
 <net name="PD4" class="0">
@@
 <label x="441.96" y="276.86" size="1.4224" layer="95" rot="R180" xref="yes"/>
 </segment>
+<segment>
+<pinref part="IC6" gate="A" pin="A5"/>
+<wire x1="365.76" y1="259.08" x2="360.68" y2="259.08" width="0.1524" layer="91"/>
+<label x="360.68" y="259.08" size="1.4224" layer="95" rot="R180" xref="yes"/>
+</segment>
 </net>
 <net name="PD5" class="0">
@@
 <label x="441.96" y="274.32" size="1.4224" layer="95" rot="R180" xref="yes"/>
 </segment>
+<segment>
+<pinref part="IC6" gate="A" pin="A6"/>
+<wire x1="365.76" y1="256.54" x2="360.68" y2="256.54" width="0.1524" layer="91"/>
+<label x="360.68" y="256.54" size="1.4224" layer="95" rot="R180" xref="yes"/>
+</segment>
 </net>
 <net name="PD6" class="0">
@@
 <label x="441.96" y="271.78" size="1.4224" layer="95" rot="R180" xref="yes"/>
 </segment>
+<segment>
+<pinref part="IC6" gate="A" pin="A7"/>
+<wire x1="365.76" y1="254" x2="360.68" y2="254" width="0.1524" layer="91"/>
+<label x="360.68" y="254" size="1.4224" layer="95" rot="R180" xref="yes"/>
+</segment>
 </net>
 <net name="PD7" class="0">
@@
 <label x="441.96" y="269.24" size="1.4224" layer="95" rot="R180" xref="yes"/>
 </segment>
+<segment>
+<pinref part="IC6" gate="A" pin="A8"/>
+<wire x1="365.76" y1="251.46" x2="360.68" y2="251.46" width="0.1524" layer="91"/>
+<label x="360.68" y="251.46" size="1.4224" layer="95" rot="R180" xref="yes"/>
+</segment>
 </net>
 <net name="/ACK" class="0">
@@
 <label x="114.3" y="144.78" size="1.4224" layer="95" rot="R90" xref="yes"/>
 </segment>
+<segment>
+<pinref part="IC6" gate="A" pin="B1"/>
+<wire x1="391.16" y1="269.24" x2="396.24" y2="269.24" width="0.1524" layer="91"/>
+<label x="396.24" y="269.24" size="1.4224" layer="95" xref="yes"/>
+</segment>
 </net>
 <net name="PD1_IN" class="0">
@@
 <label x="111.76" y="144.78" size="1.4224" layer="95" rot="R90" xref="yes"/>
 </segment>
+<segment>
+<pinref part="IC6" gate="A" pin="B2"/>
+<wire x1="391.16" y1="266.7" x2="396.24" y2="266.7" width="0.1524" layer="91"/>
+<label x="396.24" y="266.7" size="1.4224" layer="95" xref="yes"/>
+</segment>
 </net>
 <net name="PD2_IN" class="0">
@@
 <label x="109.22" y="144.78" size="1.4224" layer="95" rot="R90" xref="yes"/>
 </segment>
+<segment>
+<pinref part="IC6" gate="A" pin="B3"/>
+<wire x1="391.16" y1="264.16" x2="396.24" y2="264.16" width="0.1524" layer="91"/>
+<label x="396.24" y="264.16" size="1.4224" layer="95" xref="yes"/>
+</segment>
 </net>
 <net name="PD3_IN" class="0">
@@
 <label x="106.68" y="144.78" size="1.4224" layer="95" rot="R90" xref="yes"/>
 </segment>
+<segment>
+<pinref part="IC6" gate="A" pin="B4"/>
+<wire x1="391.16" y1="261.62" x2="396.24" y2="261.62" width="0.1524" layer="91"/>
+<label x="396.24" y="261.62" size="1.4224" layer="95" xref="yes"/>
+</segment>
 </net>
 <net name="PD4_IN" class="0">
@@
 <label x="104.14" y="144.78" size="1.4224" layer="95" rot="R90" xref="yes"/>
 </segment>
+<segment>
+<pinref part="IC6" gate="A" pin="B5"/>
+<wire x1="391.16" y1="259.08" x2="396.24" y2="259.08" width="0.1524" layer="91"/>
+<label x="396.24" y="259.08" size="1.4224" layer="95" xref="yes"/>
+</segment>
 </net>
 <net name="PD5_IN" class="0">
@@
 <label x="101.6" y="144.78" size="1.4224" layer="95" rot="R90" xref="yes"/>
 </segment>
+<segment>
+<pinref part="IC6" gate="A" pin="B6"/>
+<wire x1="391.16" y1="256.54" x2="396.24" y2="256.54" width="0.1524" layer="91"/>
+<label x="396.24" y="256.54" size="1.4224" layer="95" xref="yes"/>
+</segment>
 </net>
 <net name="PD6_IN" class="0">
@@
 <label x="99.06" y="144.78" size="1.4224" layer="95" rot="R90" xref="yes"/>
 </segment>
+<segment>
+<pinref part="IC6" gate="A" pin="B7"/>
+<wire x1="391.16" y1="254" x2="396.24" y2="254" width="0.1524" layer="91"/>
+<label x="396.24" y="254" size="1.4224" layer="95" xref="yes"/>
+</segment>
 </net>
 <net name="PD7_IN" class="0">
@@
 <label x="96.52" y="144.78" size="1.4224" layer="95" rot="R90" xref="yes"/>
 </segment>
-</net>
+<segment>
+<pinref part="IC6" gate="A" pin="B8"/>
+<wire x1="391.16" y1="251.46" x2="396.24" y2="251.46" width="0.1524" layer="91"/>
+<label x="396.24" y="251.46" size="1.4224" layer="95" xref="yes"/>
+</segment>
+</net>

Commit message: Another buffer added to printer port
Parts:
- added IC7: 74245SSOP, 74xx-eu:74245SSOP
Connections:
- removed net /STB: JP9.1
- new net /PSTB: IC7A.A8, JP9.1
- new net /PSTB_IN: IC7A.B8, U$1.RXA1/PB6
- net GND: now also IC7A.DIR, IC7A.G
Changed lines of the file:
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@@
 <part name="IC6" library="74xx-eu" deviceset="74*245" device="SSOP" value="74245SSOP"/>
 <part name="GND22" library="supply1" deviceset="GND" device=""/>
+<part name="IC7" library="74xx-eu" deviceset="74*245" device="SSOP" value="74245SSOP"/>
 </parts>
 <sheets>
@@
 <instance part="JP9" gate="A" x="454.66" y="274.32"/>
 <instance part="IC6" gate="A" x="378.46" y="256.54"/>
-<instance part="GND22" gate="1" x="363.22" y="238.76"/>
+<instance part="GND22" gate="1" x="363.22" y="198.12"/>
 <instance part="IC6" gate="P" x="15.24" y="190.5"/>
+<instance part="IC7" gate="A" x="378.46" y="215.9"/>
 </instances>
 <busses>
@@
 <wire x1="363.22" y1="246.38" x2="363.22" y2="243.84" width="0.1524" layer="91"/>
 <pinref part="IC6" gate="A" pin="G"/>
-<wire x1="363.22" y1="243.84" x2="363.22" y2="241.3" width="0.1524" layer="91"/>
+<wire x1="363.22" y1="243.84" x2="363.22" y2="205.74" width="0.1524" layer="91"/>
+<wire x1="363.22" y1="205.74" x2="363.22" y2="203.2" width="0.1524" layer="91"/>
+<wire x1="363.22" y1="203.2" x2="363.22" y2="200.66" width="0.1524" layer="91"/>
 <wire x1="365.76" y1="243.84" x2="363.22" y2="243.84" width="0.1524" layer="91"/>
 <junction x="363.22" y="243.84"/>
+<pinref part="IC7" gate="A" pin="DIR"/>
+<wire x1="365.76" y1="205.74" x2="363.22" y2="205.74" width="0.1524" layer="91"/>
+<junction x="363.22" y="205.74"/>
+<pinref part="IC7" gate="A" pin="G"/>
+<wire x1="365.76" y1="203.2" x2="363.22" y2="203.2" width="0.1524" layer="91"/>
+<junction x="363.22" y="203.2"/>
 </segment>
 </net>
@@
 </segment>
 </net>
-<net name="/STB" class="0">
+<net name="/PSTB" class="0">
 <segment>
 <pinref part="JP9" gate="A" pin="1"/>
@@
 <label x="441.96" y="289.56" size="1.4224" layer="95" rot="R180" xref="yes"/>
 </segment>
+<segment>
+<pinref part="IC7" gate="A" pin="A8"/>
+<wire x1="365.76" y1="210.82" x2="358.14" y2="210.82" width="0.1524" layer="91"/>
+<label x="358.14" y="210.82" size="1.4224" layer="95" rot="R180" xref="yes"/>
+</segment>
 </net>
 <net name="PD0" class="0">
@@
 </segment>
 </net>
+<net name="/PSTB_IN" class="0">
+<segment>
+<pinref part="U$1" gate="G$1" pin="RXA1/PB6"/>
+<wire x1="137.16" y1="86.36" x2="152.4" y2="86.36" width="0.1524" layer="91"/>
+</segment>
+<segment>
+<pinref part="IC7" gate="A" pin="B8"/>
+<wire x1="391.16" y1="210.82" x2="396.24" y2="210.82" width="0.1524" layer="91"/>
+<label x="396.24" y="210.82" size="1.4224" layer="95" xref="yes"/>
+</segment>
+</net>

Commit message: Power trace updated
Parts:
- added IC8: 74245SSOP, 74xx-eu:74245SSOP
Connections:
- new net /PRINTER_INIT_IN: IC7A.B7, U$1.TXA1/PB5
- new net /SLIN_IN: IC7A.B6, U$1.RXA0/PB4
- net /INIT: now also IC7A.A7
- net /SLIN: now also IC7A.A6
- net GND: now also IC7A.B1, IC7A.B2, IC7A.B3, IC7A.B4, IC7A.B5
Other:
- moved on the sheet: IC6, IC7

Commit message: Additional printer traces routed
Connections:
- removed net N$26: U$1.RXS//CTS1/PB7
- new net PR_OUT1: IC8A.B8, U$1.RXA0/PB4
- new net PR_OUT2: IC8A.B7, U$1.TXA0/PB3
- new net PR_OUT3: IC8A.B6, U$1./DCD0/PB2
- new net PR_OUT4: IC8A.B5, U$1./CTS0/PB1
- net /PRINTER_INIT_IN: now also U$1.RXA1/PB6; no longer U$1.TXA1/PB5
- net /PSTB_IN: now also U$1.RXS//CTS1/PB7; no longer U$1.RXA1/PB6
- net /SLIN_IN: now also U$1.TXA1/PB5; no longer U$1.RXA0/PB4
Changed lines of the file:
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@@
 <pinref part="U$1" gate="G$1" pin="CKA0//DREQ0"/>
 <wire x1="137.16" y1="91.44" x2="152.4" y2="91.44" width="0.1524" layer="91"/>
-</segment>
-</net>
-<net name="N$26" class="0">
-<segment>
-<pinref part="U$1" gate="G$1" pin="RXS//CTS1/PB7"/>
-<wire x1="137.16" y1="88.9" x2="152.4" y2="88.9" width="0.1524" layer="91"/>
+<label x="152.4" y="91.44" size="1.4224" layer="95" xref="yes"/>
 </segment>
 </net>
@@
 <net name="/PSTB_IN" class="0">
 <segment>
-<pinref part="U$1" gate="G$1" pin="RXA1/PB6"/>
-<wire x1="137.16" y1="86.36" x2="152.4" y2="86.36" width="0.1524" layer="91"/>
-</segment>
-<segment>
 <pinref part="IC7" gate="A" pin="B8"/>
 <wire x1="393.7" y1="266.7" x2="398.78" y2="266.7" width="0.1524" layer="91"/>
 <label x="398.78" y="266.7" size="1.4224" layer="95" xref="yes"/>
 </segment>
+<segment>
+<pinref part="U$1" gate="G$1" pin="RXS//CTS1/PB7"/>
+<wire x1="137.16" y1="88.9" x2="152.4" y2="88.9" width="0.1524" layer="91"/>
+<label x="152.4" y="88.9" size="1.4224" layer="95" xref="yes"/>
+</segment>
 </net>
 <net name="/PRINTER_INIT_IN" class="0">
@@
 </segment>
 <segment>
-<pinref part="U$1" gate="G$1" pin="TXA1/PB5"/>
-<wire x1="137.16" y1="83.82" x2="152.4" y2="83.82" width="0.1524" layer="91"/>
+<pinref part="U$1" gate="G$1" pin="RXA1/PB6"/>
+<wire x1="137.16" y1="86.36" x2="152.4" y2="86.36" width="0.1524" layer="91"/>
+<label x="152.4" y="86.36" size="1.4224" layer="95" xref="yes"/>
 </segment>
 </net>
@@
 </segment>
 <segment>
+<pinref part="U$1" gate="G$1" pin="TXA1/PB5"/>
+<wire x1="137.16" y1="83.82" x2="152.4" y2="83.82" width="0.1524" layer="91"/>
+<label x="152.4" y="83.82" size="1.4224" layer="95" xref="yes"/>
+</segment>
+</net>
+<net name="PR_OUT1" class="0">
+<segment>
 <pinref part="U$1" gate="G$1" pin="RXA0/PB4"/>
 <wire x1="137.16" y1="81.28" x2="152.4" y2="81.28" width="0.1524" layer="91"/>
-</segment>
-</net>
+<label x="152.4" y="81.28" size="1.4224" layer="95" xref="yes"/>
+</segment>
+<segment>
+<pinref part="IC8" gate="A" pin="B8"/>
+<wire x1="393.7" y1="223.52" x2="401.32" y2="223.52" width="0.1524" layer="91"/>
+</segment>
+</net>
+<net name="PR_OUT2" class="0">
+<segment>
+<pinref part="IC8" gate="A" pin="B7"/>
+<wire x1="393.7" y1="226.06" x2="401.32" y2="226.06" width="0.1524" layer="91"/>
+</segment>
+<segment>
+<pinref part="U$1" gate="G$1" pin="TXA0/PB3"/>
+<wire x1="137.16" y1="78.74" x2="152.4" y2="78.74" width="0.1524" layer="91"/>
+</segment>
+</net>
+<net name="PR_OUT3" class="0">
+<segment>
+<pinref part="U$1" gate="G$1" pin="/DCD0/PB2"/>
+<wire x1="137.16" y1="76.2" x2="152.4" y2="76.2" width="0.1524" layer="91"/>
+</segment>
+<segment>
+<pinref part="IC8" gate="A" pin="B6"/>
+<wire x1="393.7" y1="228.6" x2="401.32" y2="228.6" width="0.1524" layer="91"/>
+</segment>
+</net>
+<net name="PR_OUT4" class="0">
+<segment>
+<pinref part="IC8" gate="A" pin="B5"/>
+<wire x1="393.7" y1="231.14" x2="401.32" y2="231.14" width="0.1524" layer="91"/>
+</segment>
+<segment>
+<pinref part="U$1" gate="G$1" pin="/CTS0/PB1"/>
+<wire x1="137.16" y1="73.66" x2="152.4" y2="73.66" width="0.1524" layer="91"/>
+</segment>
+</net>
